File: flanck/pcb/flanck.sch (KiCad schematic (older format))
At the start: 105 parts, among them SW1 SW_PUSH, SW10 SW_PUSH, SW11 SW_PUSH, SW12 SW_PUSH, SW13 SW_PUSH, SW14 SW_PUSH, SW15 SW_PUSH, SW16 SW_PUSH, SW17 SW_PUSH, SW18 SW_PUSH, SW19 SW_PUSH, SW2 SW_PUSH, SW20 SW_PUSH, SW21 SW_PUSH, SW22 SW_PUSH, SW23 SW_PUSH, SW24 SW_PUSH, SW25 SW_PUSH, SW26 SW_PUSH, SW27 SW_PUSH, SW28 SW_PUSH, SW29 SW_PUSH, SW3 SW_PUSH, SW30 SW_PUSH, SW31 SW_PUSH, SW32 SW_PUSH, SW33 SW_PUSH, SW34 SW_PUSH, SW35 SW_PUSH, SW36 SW_PUSH, SW37 SW_PUSH, SW38 SW_PUSH, SW39 SW_PUSH, SW4 SW_PUSH, SW40 SW_PUSH, SW41 SW_PUSH, SW42 SW_PUSH, SW43 SW_PUSH, SW44 SW_PUSH, SW45 SW_PUSH, SW46 SW_PUSH, SW47 SW_PUSH, SW48 SW_PUSH, SW5 SW_PUSH, SW6 SW_PUSH, SW7 SW_PUSH, SW8 SW_PUSH, SW9 SW_PUSH, U1 ProMicro

Commit message: fix pcb mounting hole sizes
Parts:
- added H8, H9: MountingHole, kbd:M2_Threads_v2, symbol Mechanical:MountingHole
Changed lines of the file:
@@
+	1    0    0    -1
+$EndComp
+$Comp
+L Mechanical:MountingHole H8
+U 1 1 5F8D58FB
+P 2425 2525
+F 0 "H8" H 2525 2571 50  0000 L CNN
+F 1 "MountingHole" H 2525 2480 50  0000 L CNN
+F 2 "kbd:M2_Threads_v2" H 2425 2525 50  0001 C CNN
+F 3 "~" H 2425 2525 50  0001 C CNN
+	1    2425 2525
+	1    0    0    -1
+$EndComp
+$Comp
+L Mechanical:MountingHole H9
+U 1 1 5F8D5BFE
+P 3625 2525
+F 0 "H9" H 3725 2571 50  0000 L CNN
+F 1 "MountingHole" H 3725 2480 50  0000 L CNN
+F 2 "kbd:M2_Threads_v2" H 3625 2525 50  0001 C CNN
+F 3 "~" H 3625 2525 50  0001 C CNN
+	1    3625 2525
 	1    0    0    -1
 $EndComp
