File: flanck/pcb/flanck.kicad_pcb (KiCad board)
At the start: 2 copper layers, 266.7 x 76.2 mm, 105 parts, among them SW1 SW_PUSH, SW10 SW_PUSH, SW11 SW_PUSH, SW12 SW_PUSH, SW13 SW_PUSH, SW14 SW_PUSH, SW15 SW_PUSH, SW16 SW_PUSH, SW17 SW_PUSH, SW18 SW_PUSH, SW19 SW_PUSH, SW2 SW_PUSH, SW20 SW_PUSH, SW21 SW_PUSH, SW22 SW_PUSH, SW23 SW_PUSH, SW24 SW_PUSH, SW25 SW_PUSH, SW26 SW_PUSH, SW27 SW_PUSH, SW28 SW_PUSH, SW29 SW_PUSH, SW3 SW_PUSH, SW30 SW_PUSH, SW31 SW_PUSH, SW32 SW_PUSH, SW33 SW_PUSH, SW34 SW_PUSH, SW35 SW_PUSH, SW36 SW_PUSH, SW37 SW_PUSH, SW38 SW_PUSH, SW39 SW_PUSH, SW4 SW_PUSH, SW40 SW_PUSH, SW41 SW_PUSH, SW42 SW_PUSH, SW43 SW_PUSH, SW44 SW_PUSH, SW45 SW_PUSH, SW46 SW_PUSH, SW47 SW_PUSH, SW48 SW_PUSH, SW5 SW_PUSH, SW6 SW_PUSH, SW7 SW_PUSH, SW8 SW_PUSH, SW9 SW_PUSH, U1 ProMicro

Commit message: fix pcb mounting hole sizes
Parts:
- added H8: MountingHole, kbd:M2_Threads_v2, F.Cu at (130.1, 81.6)
- added H9: MountingHole, kbd:M2_Threads_v2, F.Cu at (142.8, 81.6)
- H6: moved to B.Cu
- moved RSW1 3.17 mm to (136.5, 87.2)
Routing:
- net reset: track 39.0 -> 42.2 mm
- net GND: track 57.0 -> 60.2 mm
- net col2: track 164.4 -> 165.9 mm
- net col3: track 141.1 -> 142.0 mm
Other:
- board text added: "Flanck v1.0 PCB To Nagi 2020.10.18 -- pluskid"
- board text removed: "Flanck v1.0 PCB, pluskid"

Commit message: updated drill hole size per JLCPCB feedback
Other:
- board text added: "Flanck v1.1 PCB To Nagi 2020.10.19 -- pluskid"
- board text removed: "Flanck v1.0 PCB To Nagi 2020.10.18 -- pluskid"

Commit message: tweak mod-tap behavior
Parts:
- moved D10 11.5 mm to (232.5, 44.5)
- moved D11 11.5 mm to (251.5, 44.4)
- moved D12 11.5 mm to (263.4, 42.6)
- moved D15 11.5 mm to (80.1, 63.8)
- moved D16 11.5 mm to (99.1, 63.9)
- moved D17 11.5 mm to (118.2, 63.7)
- moved D18 11.5 mm to (127.7, 61.9)
- moved D21 11.5 mm to (213.4, 63.9)
- moved D22 11.5 mm to (232.5, 63.9)
- moved D23 11.5 mm to (251.5, 63.9)
- moved D24 11.5 mm to (263.4, 62.2)
- moved D28 11.5 mm to (99.1, 83.0)
- moved D29 11.5 mm to (118.2, 82.9)
- moved D3 11.5 mm to (80.1, 44.5)
- moved D30 11.5 mm to (127.7, 81.1)
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