File: flanck/top-plate/top-plate.kicad_pcb (KiCad board)
At the start: 2 copper layers, 266.7 x 76.2 mm, 55 parts, among them SW1 SW_PUSH, SW10 SW_PUSH, SW11 SW_PUSH, SW12 SW_PUSH, SW13 SW_PUSH, SW14 SW_PUSH, SW15 SW_PUSH, SW16 SW_PUSH, SW17 SW_PUSH, SW18 SW_PUSH, SW19 SW_PUSH, SW2 SW_PUSH, SW20 SW_PUSH, SW21 SW_PUSH, SW22 SW_PUSH, SW23 SW_PUSH, SW24 SW_PUSH, SW25 SW_PUSH, SW26 SW_PUSH, SW27 SW_PUSH, SW28 SW_PUSH, SW29 SW_PUSH, SW3 SW_PUSH, SW30 SW_PUSH, SW31 SW_PUSH, SW32 SW_PUSH, SW33 SW_PUSH, SW34 SW_PUSH, SW35 SW_PUSH, SW36 SW_PUSH, SW37 SW_PUSH, SW38 SW_PUSH, SW39 SW_PUSH, SW4 SW_PUSH, SW40 SW_PUSH, SW41 SW_PUSH, SW42 SW_PUSH, SW43 SW_PUSH, SW44 SW_PUSH, SW45 SW_PUSH, SW46 SW_PUSH, SW47 SW_PUSH, SW48 SW_PUSH, SW5 SW_PUSH, SW6 SW_PUSH, SW7 SW_PUSH, SW8 SW_PUSH, SW9 SW_PUSH

Commit message: fix pcb mounting hole sizes
Other:
- outline, holes or cut-outs redrawn
Changed lines of the file:
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@@
   (general
     (thickness 1.6)
-    (drawings 8)
+    (drawings 16)
     (tracks 0)
     (zones 0)
@@
     (fp_line (start 9.525 9.525) (end 9.525 -9.525) (layer F.Fab) (width 0.15))
   )
+  (gr_line (start 147.6 36.395) (end 268.25 36.395) (layer Edge.Cuts) (width 0.2))
+  (gr_line (start 146.0125 91.9575) (end 146.0125 37.9825) (layer Edge.Cuts) (width 0.2))
+  (gr_line (start 128.55 93.545) (end 144.425 93.545) (layer Edge.Cuts) (width 0.2))
+  (gr_line (start 126.9625 37.9825) (end 126.9625 91.9575) (layer Edge.Cuts) (width 0.2))
+  (gr_arc (start 147.6 37.9825) (end 147.6 36.395) (angle -90) (layer Edge.Cuts) (width 0.2))
+  (gr_arc (start 144.425 91.9575) (end 144.425 93.545) (angle -90) (layer Edge.Cuts) (width 0.2))
+  (gr_arc (start 128.55 91.9575) (end 126.9625 91.9575) (angle -90) (layer Edge.Cuts) (width 0.2))
+  (gr_line (start 125.375 36.395) (end 4.725 36.395) (layer Edge.Cuts) (width 0.2))
+  (gr_arc (start 125.375 37.9825) (end 126.9625 37.9825) (angle -90) (layer Edge.Cuts) (width 0.2))
   (gr_line (start 4.725 112.595) (end 268.25 112.595) (layer Edge.Cuts) (width 0.2))
   (gr_line (start 3.1375 37.9825) (end 3.1375 111.0075) (layer Edge.Cuts) (width 0.2))
-  (gr_line (start 268.25 36.395) (end 4.725 36.395) (layer Edge.Cuts) (width 0.2))
   (gr_line (start 269.8375 111.0075) (end 269.8375 37.9825) (layer Edge.Cuts) (width 0.2))
   (gr_arc (start 268.25 111.0075) (end 268.25 112.595) (angle -90) (layer Edge.Cuts) (width 0.2))
